File: PCB/OpenRectangle.kicad_sch (KiCad schematic)
At the start: 54 parts, among them J1 Left Stick, J10 Modifiers, J11 C Stick, J12 Buttons, J2 Buttons, J3 Modifiers, J4 C Stick, J5 GCC Cable, J6 Extra USB, J7 USB C Connector, J8 RPI_PICO-TH, J9 Left Stick, SW1 MX_SW_HS, SW10 MX_SW_HS, SW11 MX_SW_HS, SW12 MX_SW_HS, SW13 MX_SW_HS, SW14 MX_SW_HS, SW15 MX_SW_HS, SW16 MX_SW_HS, SW17 MX_SW_HS, SW18 MX_SW_HS, SW19 MX_SW_HS, SW2 MX_SW_HS, SW20 MX_SW_HS, SW3 MX_SW_HS, SW4 MX_SW_HS, SW5 MX_SW_HS, SW6 MX_SW_HS, SW7 MX_SW_HS, SW8 MX_SW_HS, SW9 MX_SW_HS

Commit message: Updated Complete Gerber
Parts:
- D2: footprint Diode_SMD:D_0805_2012Metric -> Diode_SMD:D_SOD-123
Changed lines of the file:
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@@
       (effects (font (size 1.27 1.27)))
     )
-    (property "Footprint" "Diode_SMD:D_0805_2012Metric" (at 85.7504 21.8948 90)
+    (property "Footprint" "Diode_SMD:D_SOD-123" (at 85.7504 21.8948 90)
       (effects (font (size 1.27 1.27)) hide)
     )
